File: eagle/RoPi 2560.sch (EAGLE design)
At the start: 50 parts, among them J1 AVR_SPI_PRG_6PTH, U1 ATMEGA2560AU, U2 MAX3378EEUD, U3 L298_BRIDGE_DRIVER, U4 L298_BRIDGE_DRIVER, Y1 16M

Commit message: Removed 5V <-> 3V3 selector jumper as an ATmega2560 running at 16MHz can only be supplied 5V
Parts:
- removed JP6: (no value), pinhead:PINHD-1X3
Connections:
- removed net VCC: C12.1, C13.1, C14.1, C4.1, J1.2, JP1.VCC, JP6.2, L1.2, R1.2, U$2.1, U$2.3, U$2.5, U$2.7, U1.VCC, U1.VCC1, U1.VCC2, U1.VCC3, U2.VCC
- net 3.3V: no longer JP6.1
- net 5V: now also C12.1, C13.1, C14.1, C4.1, J1.2, JP1.VCC, L1.2, R1.2, U$2.1, U$2.3, U$2.5, U$2.7, U1.VCC, U1.VCC1, U1.VCC2, U1.VCC3, U2.VCC; no longer JP6.3
